File: 23cm-trx-kicad/23cm-trx-kicad.kicad_sch (KiCad schematic)
At the start: 67 parts, among them J1 LCD BACKLIGHT, J2 LCD I2C, Q1 BC547, Q2 BD138, Q3 BC557, SW1 RotaryEncoder_Switch, U1 ADF4153, U2 L78L09_SOT89, U3 LM741, U4 LM386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

Commit message: MC3362 symbol
Parts:
- added U5: MC3362, Package_SO:SOIC-24W_7.5x15.4mm_P1.27mm, symbol 23cm-trx-kicad-symbol-library:MC3362
Other:
- note removed: "DRAW SYMBOL FOR MC3362"
Changed lines of the file:
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@@
 	(generator "eeschema")
 	(generator_version "8.0")
-	(paper "A4")
+	(paper "A3")
 	(junction
 		(at 234.95 41.91)
@@
 	(text "23CM TRANSCEIVER"
 		(exclude_from_sim no)
-		(at 203.708 189.738 0)
+		(at 326.136 276.86 0)
 		(effects
 			(font
@@
 	(text "DRAW SYMBOL\nFOR VCO"
 		(exclude_from_sim no)
-		(at 233.172 171.704 0)
+		(at 355.6 258.826 0)
 		(effects
 			(font
@@
 		)
 	)
-	(text "DRAW SYMBOL\nFOR MC3362"
-		(exclude_from_sim no)
-		(at 270.764 171.45 0)
-		(effects
-			(font
-				(size 1.27 1.27)
-			)
-		)
-	)
 	(text "POWER\nAMPLIFIER\n(PA)"
 		(exclude_from_sim no)
@@
 	(text "PARTIAL DRAFT"
 		(exclude_from_sim no)
-		(at 276.098 193.294 0)
+		(at 398.526 280.416 0)
 		(effects
 			(font
@@
 	(text "NOTING HAMS WANT THE 1240-1300 MHz RANGE:\n\nPOSSIBLE VCOs @ 1100-1350MHz:\n - ALPS-1679C (NO RECORD) - UNOBTAINIUM\n - Y17C (GERMAN RECORD AT https://www.mikrocontroller.net/topic/353869 SUGGESTS 0.5V-9V RANGE NAVIGATES 1087-1345MHz) - UNOBTAINIUM\n\nOTHERS (GOOD):\n - M1200 (NOMINAL 1200MHz, +0-5V NAVIGATES 1150-1350MHz) - 6RMB @ https://www.fresend.com/productinfo/647892.html [CURRENT PRODUCT]\n - RFINT INNOTION YSGM 111308 (NOMINAL 1200MHz, +0.5-4.5V NAVIGATES 1100-1350MHz, THEORETICAL 1050-1400MHz RANGE) - $1.14 @ https://www.aliexpress.com/item/1005005589982171.html [MULTI VENDOR]\n - FDK IR013 (NOMINAL 1300MHz, NAVIGATES 1200-1400MHz) - $1.08 @ https://www.aliexpress.com/item/1005007461973192.html\n - UCVE1-W05A (MARKED A041; NAVIGATES 1200-1670MHz) - $0.89 @ https://www.aliexpress.com/item/1005005589963281.html or $3.20 @ https://www.aliexpress.com/item/1005007218413812.html\n - MURATA MQW540A1G40R6 (NOMINAL 1500MHz, NAVIGATES 1200-1600MHz) - $1.73 @ https://www.aliexpress.com/item/1005007376224853.html\n - MARUWA MVE-1377 (MARKED E1377; NOMINAL 1377MHZ; NAVIGATES 1200-1400MHz) - $1.73 @ https://www.aliexpress.com/item/1005007372058424.html\n - ENFVH1D2SA4 (MARKED 12 VHA4; NAVIGATES 1200-1400MHz) - $2.16 @ https://www.aliexpress.com/item/1005007376529487.html\n \nOTHERS (SKETCHY):\n - FLYSTEN FVCO1200 (NOMINAL 1200MHz, NAVIGATES 1100-1300MHz) - $4 @ https://www.aliexpress.com/item/1005006828275413.html - TOP END IFFY\n - TDK QVC811171RT-2045 (OBSOLETE; NOMINAL 1171MHz, NAVIGATES ?) - $2.59 @ https://www.aliexpress.com/item/1005006430205486.html\n\nOTHERS (NO GOOD):\n - MAX2754 (NOMINAL 1200MHz, +0.4-2.4V NAVIGATES 1145-1250MHz) - $4 @ https://www.aliexpress.com/item/32834463347.html - NO FREQUENCY MATCH\n\nOTHERS (NO SUPPLY OR INFO):\n - Alps E-D18A (1100-1400MHz)\n - Kruse Electronics 5011M2 (ANTIQUE)\n - PE1V13013 (1200-1800MHz)\n - PE1V11018 (1200-1800MHz)"
 		(exclude_from_sim no)
-		(at 302.768 41.402 0)
+		(at 124.714 246.38 0)
 		(effects
 			(font
@@
 					(unit 1)
 				)
+			)
+		)
+	)
+	(symbol
+		(lib_id "23cm-trx-kicad-symbol-library:MC3362")
+		(at 337.82 193.04 0)
+		(unit 1)
+		(exclude_from_sim no)
+		(in_bom yes)
+		(on_board yes)
+		(dnp no)
+		(fields_autoplaced yes)
+		(property "Reference" "U5"
+			(at 337.82 152.4 0)
+			(effects
+				(font
+					(size 1.27 1.27)
+				)
+			)
+		)
+		(property "Value" "MC3362"
+			(at 337.82 154.94 0)
+			(effects
+				(font
+					(size 1.27 1.27)
+				)
+			)
+		)
+		(property "Footprint" "Package_SO:SOIC-24W_7.5x15.4mm_P1.27mm"
+			(at 337.82 193.04 0)
+			(effects
+				(font
+					(size 1.27 1.27)
+				)
+				(hide yes)
+			)
+		)
+		(property "Datasheet" "https://www.discriminator.nl/ic/mc3362.pdf"
+			(at 337.82 193.04 0)
+			(effects
+				(font
+					(size 1.27 1.27)
+				)
+				(hide yes)
+			)
+		)
+		(property "Description" "Low power narrowband FM receiver."
+			(at 337.82 193.04 0)
+			(effects
+				(font
+					(size 1.27 1.27)
+				)
+				(hide yes)
+			)
+		)
+		(property "MPN" "MC3362"
+			(at 337.82 193.04 0)
+			(effects
+				(font
+					(size 1.27 1.27)
+				)
+				(hide yes)
+			)
+		)
+		(property "Manufacturer" "Motorola"
+			(at 337.82 193.04 0)
+			(effects
+				(font
+					(size 1.27 1.27)
+				)
+				(hide yes)
+			)
+		)
+		(pin "17"
+		)
+		(pin "7"
+		)
+		(pin "20"
+		)
+		(pin "10"
+		)
+		(pin "12"
+		)
+		(pin "2"
+		)
+		(pin "16"
+		)
+		(pin "18"
+		)
+		(pin "1"
+		)
+		(pin "9"
+		)
+		(pin "3"
+		)
+		(pin "22"
+		)
+		(pin "19"
+		)
+		(pin "24"
+		)
+		(pin "23"
+		)
+		(pin "15"
+		)
+		(pin "6"
+		)
+		(pin "13"
+		)
+		(pin "11"
+		)
+		(pin "14"
+		)
+		(pin "4"
+		)
+		(pin "5"
+		)
+		(pin "8"
+		)
+		(pin "21"
+		)
+		(instances
+			(project ""
+				(path "/02f64fd1-78db-4ce7-af00-a5ea9858044e"
+					(reference "U5")
+					(unit 1)
+				)
