File: 23cm-trx-kicad/23cm-trx-kicad.kicad_sch (KiCad schematic)
At the start: 68 parts, among them J1 LCD BACKLIGHT, J2 LCD I2C, Q1 BC547, Q2 BD138, Q3 BC557, SW1 RotaryEncoder_Switch, U1 ADF4153, U2 L78L09_SOT89, U3 LM741, U4 LM386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

Commit message: IF filter
Parts:
- added C25, C26: 15pF, Capacitor_SMD:C_0603_1608Metric, symbol Device:C_Small
- added C27: 1pF, Capacitor_SMD:C_0402_1005Metric, symbol Device:C_Small
- added C28: 10pF, symbol Device:C_Small
- added C29, C31: 15pF, symbol Device:C_Small
- added C30: 56pF, symbol Device:C_Small
- added L1, L2: 300nH, Inductor_SMD:L_1008_2520Metric, symbol Device:L
Connections:
- net GND: now also C25.2, C30.2, C31.2, L1.2, L2.2
- net IF-FILTERED: now reaches U5.1 (MIXER1_IN1)
- net IF-FILTERED: now also C25.1, C26.1
- new net: C26.2, C29.2, C31.1
- new net: C27.1, C28.1, L1.1
- new net: C27.2, C29.1, L2.1
- new net IF-UNFILTERED: C28.2, C30.1
Other:
- note added: "COMPONENTS IN THIS AREA ARE PRIMARILY SELECTED FOR PRECISION BUT ADDITIONALLY INDUCTORS SHOULD HAVE A LOW DC RESISTANCE (DCR) AND A HIGH CURRENT RATING AND A RELATIVELY HIGH Q RATING WITH STABLE RESPONSE ACROSS THE DESIGNED RANGE OF FREQUENCIES."
- note added: "FM RECEIVER"
- note added: "INTERMEDIATE FREQUENCY (IF) FILTER"
- moved on the sheet: U5

Commit message: More schematic work
Other:
- note added: "INTERMEDIATE FREQUENCY (IF) PASSIVE FILTER"
- note removed: "INTERMEDIATE FREQUENCY (IF) FILTER"
- moved on the sheet: C25, C26, C27, C29, C31, L1, L2

Commit message: Further schematic work
Parts:
- added C32, C33: 47uF, Capacitor_SMD:C_1206_3216Metric, symbol Device:C_Polarized_Small
- added C34: 120, Capacitor_SMD:C_0805_2012Metric, symbol Device:C_Small
- added C35, C37, C38, C39, C40: 100nF, Capacitor_SMD:C_0805_2012Metric, symbol Device:C_Small
- added C36: 47uF, Capacitor_SMD:C_1206_3216Metric, symbol Device:C_Small
- added Q4: 2SC1815, Package_TO_SOT_THT:TO-92_Inline, symbol Transistor_BJT:2SC1815
- added R24: 1.5K, Resistor_SMD:R_0805_2012Metric, symbol Device:R_Small_US
- added R25: 33K, Capacitor_SMD:C_0805_2012Metric, symbol Device:R_Small_US
- added R26: 10K, Capacitor_SMD:C_0805_2012Metric, symbol Device:R_Small_US
- added Y2: 455kHz, symbol Device:Crystal_GND3
- R20: footprint (none) -> Resistor_SMD:R_0805_2012Metric; LCSC Part # (none) -> C4310; MPN (none) -> 0805W8F1501T5E; Manufacturer (none) -> Uniroyal
- R21: footprint (none) -> Resistor_SMD:R_0805_2012Metric; LCSC Part # (none) -> C17513; MPN (none) -> 0805W8F1001T5E; Manufacturer (none) -> Uniroyal
Connections:
- net 9V: now also Q4.1 (E); no longer U2.1 (OUT)
- net GND: now also C32.2, C33.2, C34.2, C35.1, C40.1
- net at U5.10 (METER_DRIVE): now also C39.1, R25.2
- net at U5.11 (CARRIER_DETECT): now also R26.2
- net at U5.3 (LO2_EMIT): now also C34.1, C36.2
- net at U5.4 (LO2_BASE): now also C36.1
- net at U5.5 (MIXER2_OUT): now also Y2.2
- net at U5.6 (VCC): now also C35.2, C38.2, C39.2, C40.2, R25.1, R26.1, Y2.3
- net at U5.7 (LIMITER_IN): now also Y2.1
- net at U5.8 (LIMITER_DCP1): now also C37.2, C38.1
- net at U5.9 (LIMITER_DCP2): now also C37.1
- new net: C33.1, Q4.3 (B), R24.2
- new net: C32.1, Q4.2 (C), R24.1, U2.1 (OUT)
- no-connect marks 5 -> 10
Other:
- note added: "9V EMITTER FOLLOWER BUFFER / FILTER"
- note added: "CLAMPS THE SIGNAL WITHIN +/- 0.7V"
- note added: "CTCSS AND 1750MHz FILTERS"
- note added: "DRAW CRYSTAL HC-49S C11239"
- note added: "IMPROVES TRANSIENT RESPONSE AND REDUCES EXTERNAL NOISE."
- note added: "SEE ALSO docs/filter-models/ 9v-emitter-follower-buffer-filter"
- note added: "SEE ALSO docs/filter-models/ctcss-and-1750mhz-filters"
- note added: "SEE ALSO docs/filter-models/if-filter"
- note added: "THIS POTENTIOMETER PRIMARILY CONTROLS THE 1750Hz TONE VOLUME RELATIVE TO THE CTCSS TONES."
- note added: "THIS SECTION IS USED TO CONDITION MCU-BASED TONES USED FOR REPEATER COMMUNICATIONS."
- note added: "THIS WAS 12 PREVIOUSLY"
- note added: "XL4015 BASED 13.8V REGULATOR ACCEPTS 8-36V INPUT NOMINAL, REQUIRES 15V+ FOR REGULAR OPERATIONS."
- note removed: "HIGH CURRENT FOR EASY MODIFICATION."
- note removed: "MCU-ORIGINATED AUDIO"
- note removed: "NOTE PIN NUMBERS ARE MISMATCHED TO ORIGINAL PDF SCHEMATIC. ASSUME KICAD SYMBOL BUG, SINCE RESOLVED. CHECK ALL THE DATASHEETS!"
- note removed: "THIS SECTION IS USED TO FACILITATE MCU-BASED TONE GENERATION FOR GRANTING REPEATER ACCESS. IT CAN BE OMITTED FOR MAKING DIRECT COMMUNICATIONS."
- note removed: "THIS WAS 12 IN THE ORIGINAL DESIGN, BUT IT WAS MORE LOGICAL TO USE 10 HERE TO REDUCE THE COMPONENT COUNT. SHOULD EQUATE."
- note removed: "XL4015 BASED 12V REGULATOR ACCEPTS 8-36V INPUT NOMINAL, REQUIRES 15V+ FOR REGULAR OPERATIONS."
- moved on the sheet: A1, C1, C10, C11, C12, C13, C14, C15, C16, C17, C18, C19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
